File: MO6_UltrasonicDistanceSensor/MO6_UltrasonicDistanceSensor.kicad_sch (KiCad schematic)
At the start: 0 parts

Commit message: Add detector
Parts:
- added U? (x3): 74AHC2G00, symbol 74xGxx:74AHC2G00
Connections:
- new net: U?.5, U?.7
- new net Out: U?.2, U?.3
- new net ~{Reset}: U?.6
- new net ~{Set}: U?.1
Other:
- added sheet Detector (detector.kicad_sch)
- sheet oscillator ports: added Disable, out+, out-; removed none
Changed lines of the file:
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@@
 (kicad_sch (version 20230121) (generator eeschema)
   (paper "A4")
+  (junction (at 107.95 100.33) (diameter 0) (color 0 0 0 0)
+  )
+  (wire (pts (xy 107.95 77.47) (xy 107.95 85.09))
+    (stroke (width 0) (type default))
+  )
+  (wire (pts (xy 92.71 85.09) (xy 88.9 88.9))
+    (stroke (width 0) (type default))
+  )
+  (wire (pts (xy 74.93 85.09) (xy 88.9 85.09))
+    (stroke (width 0) (type default))
+  )
+  (wire (pts (xy 125.73 33.02) (xy 130.81 33.02))
+    (stroke (width 0) (type default))
+  )
+  (wire (pts (xy 107.95 88.9) (xy 107.95 100.33))
+    (stroke (width 0) (type default))
+  )
+  (wire (pts (xy 50.8 36.83) (xy 57.15 36.83))
+    (stroke (width 0) (type default))
+  )
+  (wire (pts (xy 107.95 100.33) (xy 110.49 100.33))
+    (stroke (width 0) (type default))
+  )
+  (wire (pts (xy 74.93 88.9) (xy 74.93 97.79))
+    (stroke (width 0) (type default))
+  )
+  (wire (pts (xy 74.93 88.9) (xy 88.9 88.9))
+    (stroke (width 0) (type default))
+  )
+  (wire (pts (xy 74.93 80.01) (xy 74.93 85.09))
+    (stroke (width 0) (type default))
+  )
+  (wire (pts (xy 72.39 74.93) (xy 77.47 74.93))
+    (stroke (width 0) (type default))
+  )
+  (wire (pts (xy 74.93 80.01) (xy 77.47 80.01))
+    (stroke (width 0) (type default))
+  )
+  (wire (pts (xy 105.41 100.33) (xy 107.95 100.33))
+    (stroke (width 0) (type default))
+  )
+  (wire (pts (xy 107.95 85.09) (xy 92.71 85.09))
+    (stroke (width 0) (type default))
+  )
+  (wire (pts (xy 72.39 102.87) (xy 77.47 102.87))
+    (stroke (width 0) (type default))
+  )
+  (wire (pts (xy 74.93 97.79) (xy 77.47 97.79))
+    (stroke (width 0) (type default))
+  )
+  (wire (pts (xy 105.41 77.47) (xy 107.95 77.47))
+    (stroke (width 0) (type default))
+  )
+  (wire (pts (xy 88.9 85.09) (xy 92.71 88.9))
+    (stroke (width 0) (type default))
+  )
+  (wire (pts (xy 92.71 88.9) (xy 107.95 88.9))
+    (stroke (width 0) (type default))
+  )
+  (global_label "~{Reset}" (shape input) (at 72.39 102.87 180) (fields_autoplaced)
+    (effects (font (size 1.27 1.27)) (justify right))
+    (property "Intersheetrefs" "${INTERSHEET_REFS}" (at 64.2038 102.87 0)
+      (effects (font (size 1.27 1.27)) (justify right) hide)
+    )
+  )
+  (global_label "~{Set}" (shape input) (at 72.39 74.93 180) (fields_autoplaced)
+    (effects (font (size 1.27 1.27)) (justify right))
+    (property "Intersheetrefs" "${INTERSHEET_REFS}" (at 66.381 74.93 0)
+      (effects (font (size 1.27 1.27)) (justify right) hide)
+    )
+  )
+  (global_label "~{Reset}" (shape input) (at 130.81 33.02 0) (fields_autoplaced)
+    (effects (font (size 1.27 1.27)) (justify left))
+    (property "Intersheetrefs" "${INTERSHEET_REFS}" (at 138.9962 33.02 0)
+      (effects (font (size 1.27 1.27)) (justify left) hide)
+    )
+  )
+  (global_label "~{Set}" (shape input) (at 57.15 36.83 0) (fields_autoplaced)
+    (effects (font (size 1.27 1.27)) (justify left))
+    (property "Intersheetrefs" "${INTERSHEET_REFS}" (at 63.159 36.83 0)
+      (effects (font (size 1.27 1.27)) (justify left) hide)
+    )
+  )
+  (global_label "Out" (shape input) (at 110.49 100.33 0) (fields_autoplaced)
+    (effects (font (size 1.27 1.27)) (justify left))
+    (property "Intersheetrefs" "${INTERSHEET_REFS}" (at 116.6804 100.33 0)
+      (effects (font (size 1.27 1.27)) (justify left) hide)
+    )
+  )
+  (symbol (lib_id "74xGxx:74AHC2G00") (at 45.72 88.9 0) (unit 3)
+    (in_bom yes) (on_board yes) (dnp no) (fields_autoplaced)
+    (property "Reference" "U?" (at 52.07 87.63 0)
+      (effects (font (size 1.27 1.27)) (justify left))
+    )
+    (property "Value" "74AHC2G00" (at 52.07 90.17 0)
+      (effects (font (size 1.27 1.27)) (justify left))
+    )
+    (property "Footprint" "" (at 45.72 88.9 0)
+      (effects (font (size 1.27 1.27)) hide)
+    )
+    (property "Datasheet" "https://assets.nexperia.com/documents/data-sheet/74AHC_AHCT2G00.pdf" (at 45.72 88.9 0)
+      (effects (font (size 1.27 1.27)) hide)
+    )
+    (pin "1")
+    (pin "2")
+    (pin "7")
+    (pin "3")
+    (pin "5")
+    (pin "6")
+    (pin "4")
+    (pin "8")
+    (instances
+      (project "MO6_UltrasonicDistanceSensor"
+        (path "/56fb9f7c-526c-46d4-9d85-eda8242ef960/006c8a78-f152-41de-9a44-044636956a77"
+          (reference "U?") (unit 3)
+        )
+        (path "/56fb9f7c-526c-46d4-9d85-eda8242ef960"
+          (reference "U1") (unit 3)
+        )
+      )
+    )
+  )
+  (symbol (lib_id "74xGxx:74AHC2G00") (at 92.71 77.47 0) (unit 1)
+    (in_bom yes) (on_board yes) (dnp no) (fields_autoplaced)
+    (property "Reference" "U?" (at 91.4289 67.31 0)
+      (effects (font (size 1.27 1.27)))
+    )
+    (property "Value" "74AHC2G00" (at 91.4289 69.85 0)
+      (effects (font (size 1.27 1.27)))
+    )
+    (property "Footprint" "" (at 92.71 77.47 0)
+      (effects (font (size 1.27 1.27)) hide)
+    )
+    (property "Datasheet" "https://assets.nexperia.com/documents/data-sheet/74AHC_AHCT2G00.pdf" (at 92.71 77.47 0)
+      (effects (font (size 1.27 1.27)) hide)
+    )
+    (pin "1")
+    (pin "2")
+    (pin "7")
+    (pin "3")
+    (pin "5")
+    (pin "6")
+    (pin "4")
+    (pin "8")
+    (instances
+      (project "MO6_UltrasonicDistanceSensor"
+        (path "/56fb9f7c-526c-46d4-9d85-eda8242ef960/006c8a78-f152-41de-9a44-044636956a77"
+          (reference "U?") (unit 1)
+        )
+        (path "/56fb9f7c-526c-46d4-9d85-eda8242ef960"
+          (reference "U1") (unit 1)
+        )
+      )
+    )
+  )
+  (symbol (lib_id "74xGxx:74AHC2G00") (at 92.71 100.33 0) (unit 2)
+    (in_bom yes) (on_board yes) (dnp no) (fields_autoplaced)
+    (property "Reference" "U?" (at 91.4289 90.17 0)
+      (effects (font (size 1.27 1.27)))
+    )
+    (property "Value" "74AHC2G00" (at 91.4289 92.71 0)
+      (effects (font (size 1.27 1.27)))
+    )
+    (property "Footprint" "" (at 92.71 100.33 0)
+      (effects (font (size 1.27 1.27)) hide)
+    )
+    (property "Datasheet" "https://assets.nexperia.com/documents/data-sheet/74AHC_AHCT2G00.pdf" (at 92.71 100.33 0)
+      (effects (font (size 1.27 1.27)) hide)
+    )
+    (pin "1")
+    (pin "2")
+    (pin "7")
+    (pin "3")
+    (pin "5")
+    (pin "6")
+    (pin "4")
+    (pin "8")
+    (instances
+      (project "MO6_UltrasonicDistanceSensor"
+        (path "/56fb9f7c-526c-46d4-9d85-eda8242ef960/006c8a78-f152-41de-9a44-044636956a77"
+          (reference "U?") (unit 2)
+        )
+        (path "/56fb9f7c-526c-46d4-9d85-eda8242ef960"
+          (reference "U1") (unit 2)
+        )
+      )
+    )
+  )
+  (sheet (at 101.6 25.4) (size 24.13 13.97) (fields_autoplaced)
+    (stroke (width 0.1524) (type solid))
+    (fill (color 0 0 0 0.0000))
+    (property "Sheetname" "Detector" (at 101.6 24.6884 0)
+      (effects (font (size 1.27 1.27)) (justify left bottom))
+    )
+    (property "Sheetfile" "detector.kicad_sch" (at 101.6 39.9546 0)
+      (effects (font (size 1.27 1.27)) (justify left top))
+    )
+    (pin "Sensor_in_1" input (at 101.6 31.75 180)
+      (effects (font (size 1.27 1.27)) (justify left))
+    )
+    (pin "Sensor_in_2" input (at 101.6 34.29 180)
+      (effects (font (size 1.27 1.27)) (justify left))
+    )
+    (pin "Sens_out" output (at 125.73 33.02 0)
+      (effects (font (size 1.27 1.27)) (justify right))
+    )
+    (instances
+      (project "MO6_UltrasonicDistanceSensor"
+        (path "/56fb9f7c-526c-46d4-9d85-eda8242ef960" (page "3"))
+      )
+    )
+  )
   (sheet (at 29.21 25.4) (size 21.59 13.97) (fields_autoplaced)
     (stroke (width 0.1524) (type solid))
@@
       (effects (font (size 1.27 1.27)) (justify left top))
     )
-    (instances
+    (pin "out+" output (at 50.8 31.75 0)
+      (effects (font (size 1.27 1.27)) (justify right))
+    )
+    (pin "out-" output (at 50.8 34.29 0)
+      (effects (font (size 1.27 1.27)) (justify right))
+    )
+    (pin "Disable" output (at 50.8 36.83 0)
+      (effects (font (size 1.27 1.27)) (justify right))
+    )
+    (instances

Commit message: Laatste wijzigingen toegepast
Other:
- sheet oscillator ports: added Trigger; removed none
Changed lines of the file:
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@@
     )
   )
-  (global_label "~{Reset}" (shape input) (at 130.81 33.02 0) (fields_autoplaced)
+  (global_label "~{Reset}" (shape output) (at 130.81 33.02 0) (fields_autoplaced)
     (effects (font (size 1.27 1.27)) (justify left))
     (property "Intersheetrefs" "${INTERSHEET_REFS}" (at 138.9962 33.02 0)
@@
     )
   )
-  (global_label "~{Set}" (shape input) (at 57.15 36.83 0) (fields_autoplaced)
+  (global_label "~{Set}" (shape output) (at 57.15 36.83 0) (fields_autoplaced)
     (effects (font (size 1.27 1.27)) (justify left))
     (property "Intersheetrefs" "${INTERSHEET_REFS}" (at 63.159 36.83 0)
@@
     )
   )
-  (global_label "Out" (shape input) (at 110.49 100.33 0) (fields_autoplaced)
+  (global_label "Out" (shape output) (at 110.49 100.33 0) (fields_autoplaced)
     (effects (font (size 1.27 1.27)) (justify left))
     (property "Intersheetrefs" "${INTERSHEET_REFS}" (at 116.6804 100.33 0)
@@
       (effects (font (size 1.27 1.27)) (justify right))
     )
+    (pin "Trigger" input (at 29.21 33.02 180)
+      (effects (font (size 1.27 1.27)) (justify left))
+    )
     (instances
