File: MO6_UltrasonicDistanceSensor/detector.kicad_sch (KiCad schematic)
At the start: 27 parts, among them U5 TLV2372, U6 TLV2372, U7 TLV2372

Commit message: Laatste wijzigingen toegepast
Parts:
- removed R34, R35: 560, symbol Device:R
- removed RV?: 10k, symbol Device:R_Potentiometer
- removed unit 1 of U6
Connections:
- net Signal_amplified_3 is gone; now on an unnamed net: U6.7
Other:
- note added: "Amplifier 20 dB - Lowpass filter"
- note added: "Amplifier 20dB - Highpass filter"
- note added: "Comperator"
- note added: "Referece voltage"
- note removed: "Amplifier"
- note removed: "Highpass filter"
- moved on the sheet: C3, C5, R24, R25, R28, R30, R31, R38, RV?, U5A, U5C, U6B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
