File: MO6_UltrasonicDistanceSensor/oscillator.kicad_sch (KiCad schematic)
At the start: 25 parts, among them Q1 BC547, Q2 BC547, Q3 BC547, Q4 BC547, U1 TLV2372, U2 4017, U3 74LVC1G175, U4 74LS175

Commit message: Add detector
Parts:
- removed R14: 10k, symbol Device:R
- removed U4: 74LS175, symbol 74xx:74LS175
- added Q1, Q2, Q3, Q4: BC547, Package_TO_SOT_THT:TO-92_Inline, symbol Transistor_BJT:BC547
- added R1, R10, R11, R2, R20, R5, R7, R8: 10k, symbol Device:R
- added R22, R23: 560, symbol Device:R
- renumbered Q1 to Q5, Q2 to Q6, Q3 to Q7, Q4 to Q8, R4 to R12, R8 to R13, R12 to R14, R6 to R15, R7 to R16, R9 to R17, R11 to R18, R10 to R19, R13 to R21, R2 to R4, R1 to R6, R5 to R9, U1 to U2, U2 to U3, U3 to U4
Connections:
- net Reset is gone; now on net ~{Reset}: R13.1
- net +5V: now also U4.5 (VCC), R11.1, R5.1, R8.1
- net Disable: now also U4.6 (~{CLR}), R22.2, R23.2; no longer Q8.1 (C), R21.1
- net GND: now also U4.2 (GND), Q2.3 (E), Q3.3 (E), Q4.3 (E)
- net Oscillator: now also U4.1 (C), R2.1
- net set: now also U4.3 (D), R20.2
- net ~{Reset}: now reaches U4.4 (Q)
- net ~{Reset}: now also R1.1, R20.1
- new net: Q1.1 (C), R5.2, R7.1
- new net: Q1.3 (E), Q2.1 (C)
- new net: Q2.2 (B), R2.2
- new net: Q8.1 (C), R21.1, R22.1, R23.1
- new net: Q3.1 (C), R10.1, R8.2
- new net: Q4.2 (B), R10.2
- new net: Q3.2 (B), R7.2
- new net: Q1.2 (B), R1.2
- new net out+: Q4.1 (C), R11.2
Other:
- moved on the sheet: C2, Q6, Q7, Q8, R13, R14, R15, R16, R17, R18, R19, R21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

Commit message: Laatste wijzigingen toegepast
Connections:
- net Input renamed Trigger
Other:
- note added: "Counter"
- note added: "Enable latch"
- note added: "Oscillator"
- note added: "Output stage"
- note added: "Trigger puls"
- moved on the sheet: U2B, U2C
Changed lines of the file:
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@@
     (stroke (width 0) (type default))
+  )
+  (polyline (pts (xy 135.89 101.6) (xy 135.89 106.68))
+    (stroke (width 0) (type dash))
+  )
+  (polyline (pts (xy 215.9 101.6) (xy 215.9 106.68))
+    (stroke (width 0) (type dash))
   )
   (wire (pts (xy 214.63 64.77) (xy 217.17 64.77))
@@
     (stroke (width 0) (type default))
   )
+  (polyline (pts (xy 200.66 106.68) (xy 212.09 106.68))
+    (stroke (width 0) (type dash))
+  )
   (wire (pts (xy 255.27 124.46) (xy 260.35 124.46))
     (stroke (width 0) (type default))
@@
     (stroke (width 0) (type default))
   )
+  (polyline (pts (xy 24.13 106.68) (xy 27.94 106.68))
+    (stroke (width 0) (type dash))
+  )
   (wire (pts (xy 74.93 74.93) (xy 74.93 62.23))
     (stroke (width 0) (type default))
@@
     (stroke (width 0) (type default))
   )
+  (polyline (pts (xy 133.35 106.68) (xy 135.89 106.68))
+    (stroke (width 0) (type dash))
+  )
   (wire (pts (xy 100.33 38.1) (xy 100.33 52.07))
     (stroke (width 0) (type default))
@@
     (stroke (width 0) (type default))
   )
+  (polyline (pts (xy 26.67 29.21) (xy 38.1 29.21))
+    (stroke (width 0) (type dash))
+  )
   (wire (pts (xy 99.06 133.35) (xy 99.06 167.64))
     (stroke (width 0) (type default))
@@
     (stroke (width 0) (type default))
   )
+  (polyline (pts (xy 121.92 106.68) (xy 133.35 106.68))
+    (stroke (width 0) (type dash))
+  )
   (wire (pts (xy 48.26 74.93) (xy 48.26 76.2))
     (stroke (width 0) (type default))
@@
     (stroke (width 0) (type default))
   )
+  (polyline (pts (xy 140.97 24.13) (xy 140.97 29.21))
+    (stroke (width 0) (type dash))
+  )
   (wire (pts (xy 151.13 64.77) (xy 153.67 64.77))
     (stroke (width 0) (type default))
@@
     (stroke (width 0) (type default))
   )
+  (polyline (pts (xy 12.7 106.68) (xy 24.13 106.68))
+    (stroke (width 0) (type dash))
+  )
   (wire (pts (xy 73.66 123.19) (xy 73.66 128.27))
     (stroke (width 0) (type default))
@@
     (stroke (width 0) (type default))
   )
+  (polyline (pts (xy 129.54 29.21) (xy 140.97 29.21))
+    (stroke (width 0) (type dash))
+  )
   (wire (pts (xy 45.72 59.69) (xy 52.07 59.69))
     (stroke (width 0) (type default))
@@
     (stroke (width 0) (type default))
   )
+  (polyline (pts (xy 212.09 106.68) (xy 215.9 106.68))
+    (stroke (width 0) (type dash))
+  )
   (wire (pts (xy 234.95 58.42) (xy 234.95 59.69))
     (stroke (width 0) (type default))
@@
     (stroke (width 0) (type default))
   )
+  (polyline (pts (xy 27.94 101.6) (xy 27.94 106.68))
+    (stroke (width 0) (type dash))
+  )
   (wire (pts (xy 36.83 59.69) (xy 36.83 49.53))
     (stroke (width 0) (type default))
@@
     (stroke (width 0) (type default))
   )
+  (polyline (pts (xy 38.1 24.13) (xy 38.1 29.21))
+    (stroke (width 0) (type dash))
+  )
   (wire (pts (xy 73.66 128.27) (xy 73.66 130.81))
     (stroke (width 0) (type default))
@@
   (wire (pts (xy 228.6 121.92) (xy 228.6 124.46))
     (stroke (width 0) (type default))
+  )
+  (rectangle (start 129.54 24.13) (end 273.05 95.25)
+    (stroke (width 0) (type dash))
+    (fill (type none))
+  )
+  (rectangle (start 26.67 24.13) (end 123.19 95.25)
+    (stroke (width 0) (type dash))
+    (fill (type none))
+  )
+  (rectangle (start 200.66 101.6) (end 271.78 160.02)
+    (stroke (width 0) (type dash))
+    (fill (type none))
+  )
+  (rectangle (start 121.92 101.6) (end 193.04 160.02)
+    (stroke (width 0) (type dash))
+    (fill (type none))
+  )
+  (rectangle (start 12.7 101.6) (end 116.84 176.53)
+    (stroke (width 0) (type dash))
+    (fill (type none))
+  )
+  (text "Enable latch" (at 201.93 105.41 0)
+    (effects (font (size 1.27 1.27) (thickness 0.254) bold) (justify left bottom))
+  )
+  (text "Output stage" (at 13.97 105.41 0)
+    (effects (font (size 1.27 1.27) (thickness 0.254) bold) (justify left bottom))
+  )
+  (text "Trigger puls" (at 123.19 105.41 0)
+    (effects (font (size 1.27 1.27) (thickness 0.254) bold) (justify left bottom))
+  )
+  (text "Counter\n" (at 130.81 27.94 0)
+    (effects (font (size 1.27 1.27) (thickness 0.254) bold) (justify left bottom))
+  )
+  (text "Oscillator" (at 27.94 27.94 0)
+    (effects (font (size 1.27 1.27) (thickness 0.254) bold) (justify left bottom))
   )
   (global_label "~{Reset}" (shape output) (at 260.35 124.46 0) (fields_autoplaced)
@@
     )
   )
-  (global_label "Input" (shape input) (at 132.08 142.24 180) (fields_autoplaced)
-    (effects (font (size 1.27 1.27)) (justify right))
-    (property "Intersheetrefs" "${INTERSHEET_REFS}" (at 124.3173 142.24 0)
-      (effects (font (size 1.27 1.27)) (justify right) hide)
-    )
-  )
   (global_label "Oscillator" (shape input) (at 27.94 158.75 180) (fields_autoplaced)
     (effects (font (size 1.27 1.27)) (justify right))
@@
   (hierarchical_label "out-" (shape input) (at 99.06 140.97 0) (fields_autoplaced)
     (effects (font (size 1.27 1.27)) (justify left))
+  )
+  (hierarchical_label "Trigger" (shape input) (at 132.08 142.24 180) (fields_autoplaced)
+    (effects (font (size 1.27 1.27)) (justify right))
   )
   (hierarchical_label "Disable" (shape output) (at 259.08 49.53 0) (fields_autoplaced)
@@
     )
   )
-  (symbol (lib_id "Amplifier_Operational:TLV2372") (at 59.69 25.4 0) (unit 2)
-    (in_bom yes) (on_board yes) (dnp no) (fields_autoplaced)
-    (property "Reference" "U2" (at 59.69 15.24 0)
-      (effects (font (size 1.27 1.27)))
-    )
-    (property "Value" "TLV2372" (at 59.69 17.78 0)
-      (effects (font (size 1.27 1.27)))
-    )
-    (property "Footprint" "" (at 59.69 25.4 0)
-      (effects (font (size 1.27 1.27)) hide)
-    )
-    (property "Datasheet" "http://www.ti.com/lit/ds/symlink/tlv2375.pdf" (at 59.69 25.4 0)
+  (symbol (lib_id "Amplifier_Operational:TLV2372") (at 77.47 3.81 0) (unit 2)
+    (in_bom yes) (on_board yes) (dnp no) (fields_autoplaced)
+    (property "Reference" "U2" (at 77.47 -6.35 0)
+      (effects (font (size 1.27 1.27)))
+    )
+    (property "Value" "TLV2372" (at 77.47 -3.81 0)
+      (effects (font (size 1.27 1.27)))
+    )
+    (property "Footprint" "" (at 77.47 3.81 0)
+      (effects (font (size 1.27 1.27)) hide)
+    )
+    (property "Datasheet" "http://www.ti.com/lit/ds/symlink/tlv2375.pdf" (at 77.47 3.81 0)
       (effects (font (size 1.27 1.27)) hide)
     )
@@
     )
   )
-  (symbol (lib_id "Amplifier_Operational:TLV2372") (at 24.13 69.85 0) (unit 3)
-    (in_bom yes) (on_board yes) (dnp no) (fields_autoplaced)
-    (property "Reference" "U2" (at 22.86 68.58 0)
-      (effects (font (size 1.27 1.27)) (justify left))
-    )
-    (property "Value" "TLV2372" (at 22.86 71.12 0)
-      (effects (font (size 1.27 1.27)) (justify left))
-    )
-    (property "Footprint" "" (at 24.13 69.85 0)
-      (effects (font (size 1.27 1.27)) hide)
-    )
-    (property "Datasheet" "http://www.ti.com/lit/ds/symlink/tlv2375.pdf" (at 24.13 69.85 0)
-      (effects (font (size 1.27 1.27)) hide)
-    )
+  (symbol (lib_id "Amplifier_Operational:TLV2372") (at 1.27 64.77 0) (unit 3)
+    (in_bom yes) (on_board yes) (dnp no) (fields_autoplaced)
+    (property "Reference" "U2" (at 0 63.5 0)
+      (effects (font (size 1.27 1.27)) (justify left))
+    )
+    (property "Value" "TLV2372" (at 0 66.04 0)
+      (effects (font (size 1.27 1.27)) (justify left))
+    )
+    (property "Footprint" "" (at 1.27 64.77 0)
+      (effects (font (size 1.27 1.27)) hide)
+    )
+    (property "Datasheet" "http://www.ti.com/lit/ds/symlink/tlv2375.pdf" (at 1.27 64.77 0)
+      (effects (font (size 1.27 1.27)) hide)
+    )
